Commit message: feat: add single-joint kinematics workflow

File: projects/ros2_point_robot_ws/src/point_robot_ros/urdf/point_robot.urdf (robot description, URDF)
Before this commit: robot point_robot, 2 links, 1 joints
Joints:
- joint camera_joint: axis (none) -> 0 0 1; limit (none) -> lower=-1.5708 upper=1.5708 effort=1.0 velocity=1.0; type fixed -> revolute

Commit message: feat: add ROS 2 camera and lidar workflow

File: projects/ros2_point_robot_ws/src/point_robot_ros/urdf/point_robot.urdf (robot description, URDF)
Before this commit: robot point_robot, 2 links, 1 joints
Links:
- added link camera_optical_frame
- added link laser_frame, mass 0.2; collision cylinder length=0.04 radius=0.06; visual cylinder length=0.04 radius=0.06
Joints:
- added joint camera_optical_joint: type fixed, parent camera_link, child camera_optical_frame, origin xyz=0 0 0 rpy=-1.5708 0 -1.5708
- added joint laser_joint: type fixed, parent base_link, child laser_frame, origin xyz=0.05 0 0.24 rpy=0 0 0
